File: kicad/mushi_rounded.kicad_pcb (KiCad board)
At the start: 2 copper layers, 261 x 90.8 mm, 86 parts

Commit message: separate rounded
Routing:
- net GND: track 501.2 -> 511.4 mm
- net rGND: track 520.6 -> 529.3 mm
- net matrix_pinky_top: track 127.1 -> 124.4 mm
- net matrix_ring_top: track 103.9 -> 101.3 mm
- net mirror_matrix_pinky_top: track 110.4 -> 108.4 mm
- net mirror_matrix_ring_top: track 87.5 -> 85.7 mm
- net mirror_matrix_pinky_middle: track 112.9 -> 111.1 mm
- net matrix_middle_top: track 86.0 -> 84.3 mm
- net thumbs_middle_cluster: track 74.9 -> 73.2 mm
- net matrix_ring_bottom: track 123.0 -> 124.6 mm
- net matrix_index_top: track 62.3 -> 60.9 mm
- net rRX: track 43.2 -> 42.0 mm
- net matrix_index_bottom: track 70.1 -> 69.0 mm
- net thumbs_outer_cluster: track 55.4 -> 54.2 mm
- net mirror_matrix_index_top: track 46.7 -> 45.6 mm
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