File: kicad/mushi-rounded.kicad_pcb (KiCad board)
At the start: 2 copper layers, 261 x 90.8 mm, 86 parts

Commit message: cleanup
Routing:
- net rGND: track 509.5 -> 520.6 mm
- net GND: track 490.7 -> 501.2 mm
- net mirror_matrix_ring_bottom: track 103.4 -> 111.1 mm
- net mirror_matrix_middle_bottom: track 79.3 -> 83.9 mm
- net mirror_matrix_pinky_bottom: track 133.6 -> 137.8 mm
- net mirror_matrix_index_bottom: track 56.7 -> 60.4 mm
- net mirror_thumbs_inner_cluster: track 90.4 -> 93.8 mm
- net matrix_pinky_bottom: track 150.3 -> 153.3 mm
- net mirror_matrix_outer_bottom: track 33.1 -> 36.1 mm
- net mirror_thumbs_middle_cluster: track 72.3 -> 75.0 mm
- net mirror_thumbs_outer_cluster: track 62.2 -> 64.3 mm
- net mirror_matrix_pinky_top: track 108.4 -> 110.4 mm
- net mirror_matrix_ring_middle: track 86.8 -> 88.8 mm
- net mirror_matrix_ring_top: track 85.6 -> 87.5 mm
- net rP3V3: track 37.3 -> 39.2 mm
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
Commit message: improve rounded
Routing:
- net mirror_matrix_pinky_top: track 110.4 -> 127.0 mm
- net mirror_matrix_middle_top: track 70.0 -> 82.7 mm
- net mirror_matrix_ring_top: track 87.5 -> 96.8 mm
- net mirror_matrix_index_top: track 46.7 -> 54.7 mm
- net mirror_matrix_middle_middle: track 69.7 -> 77.2 mm
- net mirror_matrix_ring_middle: track 88.8 -> 96.0 mm
- net mirror_matrix_pinky_middle: track 112.9 -> 119.5 mm
- net mirror_matrix_index_middle: track 44.9 -> 50.6 mm
- net mirror_matrix_outer_middle: track 23.3 -> 27.7 mm
- net mirror_matrix_outer_top: track 28.2 -> 30.1 mm
- net mirror_thumbs_inner_cluster: track 93.8 -> 95.6 mm
- net mirror_matrix_index_bottom: track 60.4 -> 61.8 mm
- net mirror_matrix_middle_bottom: track 83.9 -> 85.2 mm
- net mirror_matrix_pinky_bottom: track 137.8 -> 139.1 mm
- net mirror_thumbs_middle_cluster: track 75.0 -> 76.1 mm
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