File: kicad/mushi.kicad_pcb (KiCad board)
At the start: 2 copper layers, 262.6 x 94.5 mm, 76 parts

Commit message: fix nets
Parts:
- removed ? (x2): , Connector_FFC-FPC:Hirose_FH12-12S-0.5SH_1x12-1MP_P0.50mm_Horizontal
- removed ? (x2): , footprints:HRO-TYPE-C-31-M-12
- added REF**: HRO-TYPE-C-31-M-12, footprints:HRO-TYPE-C-31-M-12, F.Cu at (207.1, 22.1)
- added REF**: HRO-TYPE-C-31-M-12, footprints:HRO-TYPE-C-31-M-12, F.Cu at (88.0, 22.1)
- added REF**: Hirose_FH12-12S-0.5SH_1x12-1MP_P0.50mm_Horizontal, Connector_FFC-FPC:Hirose_FH12-12S-0.5SH_1x12-1MP_P0.50mm_Horizontal, F.Cu at (109.1, 65.2)
- added REF**: Hirose_FH12-12S-0.5SH_1x12-1MP_P0.50mm_Horizontal, Connector_FFC-FPC:Hirose_FH12-12S-0.5SH_1x12-1MP_P0.50mm_Horizontal, F.Cu at (186.1, 65.2)
Connections:
- net middle_cluster renamed inner_bottom
- net outer_cluster renamed outer_bottom
- D14 pad 2: middle_top -> inner_top
- D17 pad 2: (no net) -> mirror_pinky_bottom
- D18 pad 2: (no net) -> mirror_pinky_middle
- D19 pad 2: (no net) -> mirror_pinky_top
- D20 pad 2: (no net) -> mirror_ring_bottom
- D21 pad 2: (no net) -> mirror_ring_middle
- D22 pad 2: (no net) -> mirror_ring_top
- D23 pad 2: (no net) -> mirror_middle_bottom
- D24 pad 2: (no net) -> mirror_middle_middle
- D25 pad 2: (no net) -> mirror_middle_top
- D26 pad 2: (no net) -> mirror_index_bottom
- D27 pad 2: (no net) -> mirror_index_middle
- D28 pad 2: (no net) -> mirror_index_top
- D29 pad 1: (no net) -> rGP28
- D29 pad 2: (no net) -> mirror_inner_bottom
- D30 pad 1: (no net) -> rGP29
- D30 pad 2: (no net) -> mirror_inner_top
- D31 pad 1: (no net) -> rGP28
- D31 pad 2: (no net) -> mirror_outer_bottom
- D32 pad 1: (no net) -> rGP29
- D32 pad 2: (no net) -> mirror_outer_top
- S14 pad 2: middle_top -> inner_top
- S17 pad 2: (no net) -> mirror_pinky_bottom
- S18 pad 2: (no net) -> mirror_pinky_middle
- S19 pad 2: (no net) -> mirror_pinky_top
- S20 pad 2: (no net) -> mirror_ring_bottom
- S21 pad 2: (no net) -> mirror_ring_middle
- S22 pad 2: (no net) -> mirror_ring_top
- S23 pad 2: (no net) -> mirror_middle_bottom
- S24 pad 2: (no net) -> mirror_middle_middle
- S25 pad 2: (no net) -> mirror_middle_top
- S26 pad 2: (no net) -> mirror_index_bottom
- S27 pad 2: (no net) -> mirror_index_middle
- S28 pad 2: (no net) -> mirror_index_top
- S29 pad 1: rGP28 -> rGP11
- S29 pad 2: (no net) -> mirror_inner_bottom
- S30 pad 1: rGP29 -> rGP11
- S30 pad 2: (no net) -> mirror_inner_top
- S31 pad 1: rGP28 -> rGP12
- S31 pad 2: (no net) -> mirror_outer_bottom
- S32 pad 1: rGP29 -> rGP12
- S32 pad 2: (no net) -> mirror_outer_top
Routing:
- net lGP11: track 148.7 -> 0.00 mm, vias 5 -> 0
- net lGP9: track 145.8 -> 0.00 mm, vias 3 -> 0
- net lGP27: track 138.9 -> 0.00 mm, vias 1 -> 0
- net lGP12: track 137.8 -> 0.00 mm, vias 2 -> 0
- net lGP10: track 126.2 -> 0.00 mm, vias 2 -> 0
- net lGP26: track 121.1 -> 0.00 mm, vias 1 -> 0
- net lGP15: track 103.3 -> 0.00 mm, vias 1 -> 0
- net lGP28: track 91.2 -> 0.00 mm, vias 1 -> 0
- net lGP29: track 77.2 -> 0.00 mm
- net lGP3: track 39.6 -> 0.00 mm
- net lGP4: track 38.8 -> 0.00 mm
- net lGP5: track 36.4 -> 0.00 mm
- net lGP2: track 35.8 -> 0.00 mm, vias 2 -> 0
- net lGP0: track 35.7 -> 0.00 mm, vias 2 -> 0
- net lGP1: track 35.5 -> 0.00 mm, vias 2 -> 0
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- removed copper zone on B.Cu, net lGND

Commit message: fix net
Connections:
- REF** pad 2: rP3V3 -> rGND
Changed lines of the file:
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@@
 			(size 0.3 1.3)
 			(layers "F.Cu" "F.Paste" "F.Mask")
-			(net 67 "rP3V3")
+			(net 66 "rGND")
 		)
 		(pad "3" smd rect

Commit message: route left
Routing:
- net lGP9: track 0.00 -> 145.7 mm, vias 0 -> 1
- net lGP27: track 0.00 -> 145.3 mm, vias 0 -> 2
- net lGP11: track 0.00 -> 144.5 mm, vias 0 -> 2
- net lGP12: track 0.00 -> 134.8 mm, vias 0 -> 2
- net lGP26: track 0.00 -> 127.4 mm, vias 0 -> 2
- net lGP10: track 0.00 -> 119.8 mm, vias 0 -> 1
- net lGP15: track 0.00 -> 116.3 mm
- net lGP28: track 0.00 -> 96.7 mm, vias 0 -> 1
- net lGP29: track 0.00 -> 82.0 mm, vias 0 -> 1
- net rGP12: track 0.00 -> 59.0 mm
- net rGP11: track 0.00 -> 58.9 mm
- net lGP3: track 0.00 -> 50.5 mm, vias 0 -> 2
- net lGP2: track 0.00 -> 44.2 mm, vias 0 -> 2
- net lGP4: track 0.00 -> 42.4 mm, vias 0 -> 2
- net rGP10: track 0.00 -> 40.8 mm
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- added copper zone on B.Cu, net lGND

Commit message: route right
Routing:
- net rGP27: track 8.77 -> 149.5 mm, vias 0 -> 1
- net rGP26: track 8.77 -> 132.3 mm, vias 0 -> 2
- net rGP15: track 8.77 -> 121.2 mm
- net rGP9: track 37.9 -> 143.5 mm, vias 0 -> 4
- net rGP28: track 4.68 -> 106.9 mm, vias 0 -> 1
- net rGP29: track 4.68 -> 88.8 mm, vias 0 -> 2
- net rGP11: track 58.9 -> 129.7 mm, vias 0 -> 2
- net rGP10: track 40.8 -> 107.7 mm, vias 0 -> 2
- net rGP12: track 59.0 -> 125.7 mm, vias 0 -> 4
- net rP3V3: track 0.00 -> 44.1 mm, vias 0 -> 1
- net rGP2: track 0.00 -> 44.1 mm, vias 0 -> 1
- net rGP3: track 0.00 -> 42.0 mm, vias 0 -> 1
- net rP5V: track 0.00 -> 37.0 mm
- net rGP4: track 0.00 -> 36.7 mm, vias 0 -> 1
- net rGP5: track 0.00 -> 33.7 mm, vias 0 -> 1
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- added copper zone on B.Cu, net rGND

Commit message: cleanup
Routing:
- net lGP3: track 50.5 -> 46.2 mm
- net lGP26: track 127.4 -> 124.7 mm
- net rGP9: track 143.5 -> 141.5 mm
- net rGP10: track 107.7 -> 106.2 mm
- net rP3V3: track 44.1 -> 45.3 mm
- net lGP10: track 119.8 -> 120.9 mm
- net rGP3: track 42.0 -> 43.0 mm
- net rGP2: track 44.1 -> 45.1 mm
- net lGP27: track 145.3 -> 144.4 mm
- net rGP26: track 132.3 -> 131.5 mm
- net rGP4: track 36.7 -> 37.5 mm
- net lGP15: track 116.3 -> 115.5 mm
- net rGP29: track 88.8 -> 88.2 mm
- net rGP15: track 121.2 -> 120.7 mm

Commit message: cleanup
Routing:
- net lGP11: track 144.5 -> 143.7 mm
- net lGP15: track 115.5 -> 114.8 mm
- net lGP26: track 124.7 -> 124.0 mm

Commit message: cleanup
Routing:
- net rGP28: track 106.7 -> 103.4 mm, vias 1 -> 0
- net lGP4: track 42.6 -> 39.9 mm, vias 2 -> 1
- net rP3V3: track 45.3 -> 47.7 mm
- net lGP2: track 44.2 -> 45.9 mm, vias 2 -> 1
- net lGP26: track 124.0 -> 124.6 mm
- net lGP15: track 114.8 -> 114.3 mm
- net lGP3: track 46.2 -> 45.9 mm, vias 2 -> 1
- net rGP29: track 88.2 -> 88.4 mm, vias 2 -> 1
- net lGP5: vias 2 -> 1

Commit message: cleanup
Routing:
- net lGP29: track 81.8 -> 84.6 mm
- net lGP27: track 144.4 -> 147.0 mm, vias 2 -> 1
- net lGP10: track 120.9 -> 122.3 mm
- net lGP9: track 145.3 -> 144.1 mm
- net lGP28: track 96.6 -> 96.1 mm, vias 1 -> 0
- net lGP26: track 124.6 -> 124.3 mm, vias 2 -> 1
